Commit message: Fixed wrong scaling/file names inside urdf file

File: tbotros_description/desc/tetherbot/tetherbot.urdf (robot description, URDF)
Before this commit: robot tetherbot0, 95 links, 94 joints
Links:
- link trianglemesh0: geometry visual mesh filename=package://tbotros_description/desc/trianglemesh0.stl scale=1 1 1
- link trianglemesh1: geometry visual mesh filename=package://tbotros_description/desc/trianglemesh1.stl scale=1 1 1
- link trianglemesh10: geometry visual mesh filename=package://tbotros_description/desc/trianglemesh10.stl scale=1 1 1
- link trianglemesh11: geometry visual mesh filename=package://tbotros_description/desc/trianglemesh11.stl scale=1 1 1
- link trianglemesh12: geometry visual mesh filename=package://tbotros_description/desc/trianglemesh12.stl scale=1 1 1
- link trianglemesh13: geometry visual mesh filename=package://tbotros_description/desc/trianglemesh13.stl scale=1 1 1
- link trianglemesh14: geometry visual mesh filename=package://tbotros_description/desc/trianglemesh14.stl scale=1 1 1
- link trianglemesh15: geometry visual mesh filename=package://tbotros_description/desc/trianglemesh15.stl scale=1 1 1
- link trianglemesh2: geometry visual mesh filename=package://tbotros_description/desc/trianglemesh2.stl scale=1 1 1
- link trianglemesh3: geometry visual mesh filename=package://tbotros_description/desc/trianglemesh3.stl scale=1 1 1
- link trianglemesh4: geometry visual mesh filename=package://tbotros_description/desc/trianglemesh4.stl scale=1 1 1
- link trianglemesh5: geometry visual mesh filename=package://tbotros_description/desc/trianglemesh5.stl scale=1 1 1
- link trianglemesh6: geometry visual mesh filename=package://tbotros_description/desc/trianglemesh6.stl scale=1 1 1
- link trianglemesh7: geometry visual mesh filename=package://tbotros_description/desc/trianglemesh7.stl scale=1 1 1
- link trianglemesh8: geometry visual mesh filename=package://tbotros_description/desc/trianglemesh8.stl scale=1 1 1
- link trianglemesh9: geometry visual mesh filename=package://tbotros_description/desc/trianglemesh9.stl scale=1 1 1

Commit message: Modified tetherbot description

File: tbotros_description/desc/tetherbot/tetherbot.urdf (robot description, URDF)
Before this commit: robot tetherbot0, 95 links, 94 joints
Links:
- added link grippoint10; visual sphere radius=0.01
- added link grippoint11; visual sphere radius=0.01
- added link grippoint12; visual sphere radius=0.01
- added link grippoint13; visual sphere radius=0.01
- added link grippoint14; visual sphere radius=0.01
- added link hold5
- added link hold6
- added link hold7
- added link hold8
- added link hold9
- added link hoverpoint10; visual sphere radius=0.01
- added link hoverpoint11; visual sphere radius=0.01
- added link hoverpoint12; visual sphere radius=0.01
- added link hoverpoint13; visual sphere radius=0.01
- added link hoverpoint14; visual sphere radius=0.01
- added link point16; visual sphere radius=0.01
- added link point17; visual sphere radius=0.01
- added link point18; visual sphere radius=0.01
- added link point19; visual sphere radius=0.01
- added link point20; visual sphere radius=0.01
- added link trianglemesh16; visual mesh filename=package://ros2_tetherbot/urdf/trianglemesh16.stl scale=1 1 1
- added link trianglemesh17; visual mesh filename=package://ros2_tetherbot/urdf/trianglemesh17.stl scale=1 1 1
- added link trianglemesh18; visual mesh filename=package://ros2_tetherbot/urdf/trianglemesh18.stl scale=1 1 1
- added link trianglemesh19; visual mesh filename=package://ros2_tetherbot/urdf/trianglemesh19.stl scale=1 1 1
- added link trianglemesh20; visual mesh filename=package://ros2_tetherbot/urdf/trianglemesh20.stl scale=1 1 1
- link trianglemesh0: geometry visual mesh filename=package://ros2_tetherbot/urdf/trianglemesh0.stl scale=1 1 1
- link trianglemesh1: geometry visual mesh filename=package://ros2_tetherbot/urdf/trianglemesh1.stl scale=1 1 1
- link trianglemesh10: geometry visual mesh filename=package://ros2_tetherbot/urdf/trianglemesh10.stl scale=1 1 1
- link trianglemesh11: geometry visual mesh filename=package://ros2_tetherbot/urdf/trianglemesh11.stl scale=1 1 1
- link trianglemesh12: geometry visual mesh filename=package://ros2_tetherbot/urdf/trianglemesh12.stl scale=1 1 1
- link trianglemesh13: geometry visual mesh filename=package://ros2_tetherbot/urdf/trianglemesh13.stl scale=1 1 1
- link trianglemesh14: geometry visual mesh filename=package://ros2_tetherbot/urdf/trianglemesh14.stl scale=1 1 1
- link trianglemesh15: geometry visual mesh filename=package://ros2_tetherbot/urdf/trianglemesh15.stl scale=1 1 1
- link trianglemesh2: geometry visual mesh filename=package://ros2_tetherbot/urdf/trianglemesh2.stl scale=1 1 1
- link trianglemesh3: geometry visual mesh filename=package://ros2_tetherbot/urdf/trianglemesh3.stl scale=1 1 1
- link trianglemesh4: geometry visual mesh filename=package://ros2_tetherbot/urdf/trianglemesh4.stl scale=1 1 1
- link trianglemesh5: geometry visual mesh filename=package://ros2_tetherbot/urdf/trianglemesh5.stl scale=1 1 1
- link trianglemesh6: geometry visual mesh filename=package://ros2_tetherbot/urdf/trianglemesh6.stl scale=1 1 1
- link trianglemesh7: geometry visual mesh filename=package://ros2_tetherbot/urdf/trianglemesh7.stl scale=1 1 1
- link trianglemesh8: geometry visual mesh filename=package://ros2_tetherbot/urdf/trianglemesh8.stl scale=1 1 1
- link trianglemesh9: geometry visual mesh filename=package://ros2_tetherbot/urdf/trianglemesh9.stl scale=1 1 1
Joints:
- removed joint gripper0_to_grippoint5
- removed joint gripper0_to_hoverpoint5
- removed joint gripper0_to_trianglemesh11
- removed joint gripper1_to_grippoint6
- removed joint gripper1_to_hoverpoint6
- removed joint gripper1_to_trianglemesh12
- removed joint gripper2_to_grippoint7
- removed joint gripper2_to_hoverpoint7
- removed joint gripper2_to_trianglemesh13
- removed joint gripper3_to_grippoint8
- removed joint gripper3_to_hoverpoint8
- removed joint gripper3_to_trianglemesh14
- removed joint gripper4_to_grippoint9
- removed joint gripper4_to_hoverpoint9
- removed joint gripper4_to_trianglemesh15
- removed joint platform0_to_trianglemesh10
- removed joint prismaticlink0_to_trianglemesh7
- removed joint prismaticlink1_to_trianglemesh8
- removed joint revolutelink0_to_trianglemesh6
- removed joint rpparm0_to_trianglemesh9
- removed joint wall0_to_trianglemesh5
- added joint gripper0_to_grippoint10: type fixed, parent gripper0, child grippoint10, origin xyz=0.0 0.0 0.029 rpy=0.0 -0.0 0.0
- added joint gripper0_to_hoverpoint10: type fixed, parent gripper0, child hoverpoint10, origin xyz=0.0 0.0 0.153 rpy=0.0 -0.0 0.0
- added joint gripper0_to_trianglemesh16: type fixed, parent gripper0, child trianglemesh16, origin xyz=0.0 0.0 0.0 rpy=0.0 -0.0 0.0
- added joint gripper1_to_grippoint11: type fixed, parent gripper1, child grippoint11, origin xyz=0.0 0.0 0.029 rpy=0.0 -0.0 0.0
- added joint gripper1_to_hoverpoint11: type fixed, parent gripper1, child hoverpoint11, origin xyz=0.0 0.0 0.153 rpy=0.0 -0.0 0.0
- added joint gripper1_to_trianglemesh17: type fixed, parent gripper1, child trianglemesh17, origin xyz=0.0 0.0 0.0 rpy=0.0 -0.0 0.0
- added joint gripper2_to_grippoint12: type fixed, parent gripper2, child grippoint12, origin xyz=0.0 0.0 0.029 rpy=0.0 -0.0 0.0
- added joint gripper2_to_hoverpoint12: type fixed, parent gripper2, child hoverpoint12, origin xyz=0.0 0.0 0.153 rpy=0.0 -0.0 0.0
- added joint gripper2_to_trianglemesh18: type fixed, parent gripper2, child trianglemesh18, origin xyz=0.0 0.0 0.0 rpy=0.0 -0.0 0.0
- added joint gripper3_to_grippoint13: type fixed, parent gripper3, child grippoint13, origin xyz=0.0 0.0 0.029 rpy=0.0 -0.0 0.0
- added joint gripper3_to_hoverpoint13: type fixed, parent gripper3, child hoverpoint13, origin xyz=0.0 0.0 0.153 rpy=0.0 -0.0 0.0
- added joint gripper3_to_trianglemesh19: type fixed, parent gripper3, child trianglemesh19, origin xyz=0.0 0.0 0.0 rpy=0.0 -0.0 0.0
- added joint gripper4_to_grippoint14: type fixed, parent gripper4, child grippoint14, origin xyz=0.0 0.0 0.029 rpy=0.0 -0.0 0.0
- added joint gripper4_to_hoverpoint14: type fixed, parent gripper4, child hoverpoint14, origin xyz=0.0 0.0 0.153 rpy=0.0 -0.0 0.0
- added joint gripper4_to_trianglemesh20: type fixed, parent gripper4, child trianglemesh20, origin xyz=0.0 0.0 0.0 rpy=0.0 -0.0 0.0
- added joint hold5_to_grippoint5: type fixed, parent hold5, child grippoint5, origin xyz=0.0 0.0 0.029 rpy=0.0 -0.0 0.0
- added joint hold5_to_hoverpoint5: type fixed, parent hold5, child hoverpoint5, origin xyz=0.0 0.0 0.039 rpy=0.0 -0.0 0.0
- added joint hold5_to_trianglemesh5: type fixed, parent hold5, child trianglemesh5, origin xyz=0.0 0.0 0.0 rpy=0.0 -0.0 0.0
- added joint hold6_to_grippoint6: type fixed, parent hold6, child grippoint6, origin xyz=0.0 0.0 0.029 rpy=0.0 -0.0 0.0
- added joint hold6_to_hoverpoint6: type fixed, parent hold6, child hoverpoint6, origin xyz=0.0 0.0 0.039 rpy=0.0 -0.0 0.0
- added joint hold6_to_trianglemesh6: type fixed, parent hold6, child trianglemesh6, origin xyz=0.0 0.0 0.0 rpy=0.0 -0.0 0.0
- added joint hold7_to_grippoint7: type fixed, parent hold7, child grippoint7, origin xyz=0.0 0.0 0.029 rpy=0.0 -0.0 0.0
- added joint hold7_to_hoverpoint7: type fixed, parent hold7, child hoverpoint7, origin xyz=0.0 0.0 0.039 rpy=0.0 -0.0 0.0
- added joint hold7_to_trianglemesh7: type fixed, parent hold7, child trianglemesh7, origin xyz=0.0 0.0 0.0 rpy=0.0 -0.0 0.0
- added joint hold8_to_grippoint8: type fixed, parent hold8, child grippoint8, origin xyz=0.0 0.0 0.029 rpy=0.0 -0.0 0.0
- added joint hold8_to_hoverpoint8: type fixed, parent hold8, child hoverpoint8, origin xyz=0.0 0.0 0.039 rpy=0.0 -0.0 0.0
- added joint hold8_to_trianglemesh8: type fixed, parent hold8, child trianglemesh8, origin xyz=0.0 0.0 0.0 rpy=0.0 -0.0 0.0
- added joint hold9_to_grippoint9: type fixed, parent hold9, child grippoint9, origin xyz=0.0 0.0 0.029 rpy=0.0 -0.0 0.0
- added joint hold9_to_hoverpoint9: type fixed, parent hold9, child hoverpoint9, origin xyz=0.0 0.0 0.039 rpy=0.0 -0.0 0.0
- added joint hold9_to_trianglemesh9: type fixed, parent hold9, child trianglemesh9, origin xyz=0.0 0.0 0.0 rpy=0.0 -0.0 0.0
- added joint platform0_to_trianglemesh15: type fixed, parent platform0, child trianglemesh15, origin xyz=0.0 0.0 0.0 rpy=0.0 -0.0 0.0
- added joint prismaticlink0_to_trianglemesh12: type fixed, parent prismaticlink0, child trianglemesh12, origin xyz=0.0 0.0 0.0 rpy=0.0 -0.0 0.0
- added joint prismaticlink1_to_trianglemesh13: type fixed, parent prismaticlink1, child trianglemesh13, origin xyz=0.0 0.0 0.0 rpy=0.0 -0.0 0.0
- added joint revolutelink0_to_trianglemesh11: type fixed, parent revolutelink0, child trianglemesh11, origin xyz=0.0 0.0 0.0 rpy=0.0 -0.0 0.0
- added joint rpparm0_to_trianglemesh14: type fixed, parent rpparm0, child trianglemesh14, origin xyz=0.0 0.0 0.0 rpy=0.0 -0.0 0.0
- added joint trianglemesh16_to_point16: type fixed, parent trianglemesh16, child point16, origin xyz=0.0 0.0 0.0 rpy=0.0 -0.0 0.0
- added joint trianglemesh17_to_point17: type fixed, parent trianglemesh17, child point17, origin xyz=0.0 0.0 0.0 rpy=0.0 -0.0 0.0
- added joint trianglemesh18_to_point18: type fixed, parent trianglemesh18, child point18, origin xyz=0.0 0.0 0.0 rpy=0.0 -0.0 0.0
- added joint trianglemesh19_to_point19: type fixed, parent trianglemesh19, child point19, origin xyz=0.0 0.0 0.0 rpy=0.0 -0.0 0.0
- added joint trianglemesh20_to_point20: type fixed, parent trianglemesh20, child point20, origin xyz=0.0 0.0 0.0 rpy=0.0 -0.0 0.0
- added joint wall0_to_hold5: type fixed, parent wall0, child hold5, origin xyz=0.527 1.585 0.002 rpy=0.0 -0.0 0.0
- added joint wall0_to_hold6: type fixed, parent wall0, child hold6, origin xyz=0.827 1.285 0.002 rpy=0.0 -0.0 0.0
- added joint wall0_to_hold7: type fixed, parent wall0, child hold7, origin xyz=0.827 0.385 0.002 rpy=0.0 -0.0 0.0
- added joint wall0_to_hold8: type fixed, parent wall0, child hold8, origin xyz=0.077 0.535 0.002 rpy=0.0 -0.0 0.0
- added joint wall0_to_hold9: type fixed, parent wall0, child hold9, origin xyz=0.077 1.435 0.002 rpy=0.0 -0.0 0.0
- added joint wall0_to_trianglemesh10: type fixed, parent wall0, child trianglemesh10, origin xyz=0.0 0.0 0.0 rpy=0.0 -0.0 0.0
- joint map_to_platform0: origin xyz=0.423 1.02 0.068 rpy=0.0 -0.0 1.5707963267948966 -> xyz=0.423 0.82 0.068 rpy=0.0 -0.0 1.5707963267948966
- joint prismaticlink0_to_prismaticlink1: origin xyz=0.0 0.0 0.2 rpy=0.0 -0.0 0.0 -> xyz=0.0 0.0 0.198 rpy=0.0 -0.0 0.0
- joint wall0_to_hold0: origin xyz=0.527 1.585 0.002 rpy=0.0 -0.0 0.0 -> xyz=0.527 1.285 0.002 rpy=0.0 -0.0 0.0
- joint wall0_to_hold1: origin xyz=0.827 1.285 0.002 rpy=0.0 -0.0 0.0 -> xyz=0.827 0.985 0.002 rpy=0.0 -0.0 0.0
- joint wall0_to_hold2: origin xyz=0.827 0.385 0.002 rpy=0.0 -0.0 0.0 -> xyz=0.827 0.185 0.002 rpy=0.0 -0.0 0.0
- joint wall0_to_hold3: origin xyz=0.077 0.535 0.002 rpy=0.0 -0.0 0.0 -> xyz=0.077 0.235 0.002 rpy=0.0 -0.0 0.0
- joint wall0_to_hold4: origin xyz=0.077 1.435 0.002 rpy=0.0 -0.0 0.0 -> xyz=0.077 1.135 0.002 rpy=0.0 -0.0 0.0

Commit message: Modified tetherbot description

File: tbotros_description/desc/tetherbot/tetherbot.urdf (robot description, URDF)
Before this commit: robot tetherbot0, 120 links, 119 joints
Links:
- link trianglemesh0: geometry visual mesh filename=package://tbotros_description/desc//trianglemesh0.stl scale=1 1 1
- link trianglemesh1: geometry visual mesh filename=package://tbotros_description/desc//trianglemesh1.stl scale=1 1 1
- link trianglemesh10: geometry visual mesh filename=package://tbotros_description/desc//trianglemesh10.stl scale=1 1 1
- link trianglemesh11: geometry visual mesh filename=package://tbotros_description/desc//trianglemesh11.stl scale=1 1 1
- link trianglemesh12: geometry visual mesh filename=package://tbotros_description/desc//trianglemesh12.stl scale=1 1 1
- link trianglemesh13: geometry visual mesh filename=package://tbotros_description/desc//trianglemesh13.stl scale=1 1 1
- link trianglemesh14: geometry visual mesh filename=package://tbotros_description/desc//trianglemesh14.stl scale=1 1 1
- link trianglemesh15: geometry visual mesh filename=package://tbotros_description/desc//trianglemesh15.stl scale=1 1 1
- link trianglemesh16: geometry visual mesh filename=package://tbotros_description/desc//trianglemesh16.stl scale=1 1 1
- link trianglemesh17: geometry visual mesh filename=package://tbotros_description/desc//trianglemesh17.stl scale=1 1 1
- link trianglemesh18: geometry visual mesh filename=package://tbotros_description/desc//trianglemesh18.stl scale=1 1 1
- link trianglemesh19: geometry visual mesh filename=package://tbotros_description/desc//trianglemesh19.stl scale=1 1 1
- link trianglemesh2: geometry visual mesh filename=package://tbotros_description/desc//trianglemesh2.stl scale=1 1 1
- link trianglemesh20: geometry visual mesh filename=package://tbotros_description/desc//trianglemesh20.stl scale=1 1 1
- link trianglemesh3: geometry visual mesh filename=package://tbotros_description/desc//trianglemesh3.stl scale=1 1 1
- link trianglemesh4: geometry visual mesh filename=package://tbotros_description/desc//trianglemesh4.stl scale=1 1 1
- link trianglemesh5: geometry visual mesh filename=package://tbotros_description/desc//trianglemesh5.stl scale=1 1 1
- link trianglemesh6: geometry visual mesh filename=package://tbotros_description/desc//trianglemesh6.stl scale=1 1 1
- link trianglemesh7: geometry visual mesh filename=package://tbotros_description/desc//trianglemesh7.stl scale=1 1 1
- link trianglemesh8: geometry visual mesh filename=package://tbotros_description/desc//trianglemesh8.stl scale=1 1 1
- link trianglemesh9: geometry visual mesh filename=package://tbotros_description/desc//trianglemesh9.stl scale=1 1 1

Commit message: Updated description

File: tbotros_description/desc/tetherbot/tetherbot.urdf (robot description, URDF)
Before this commit: robot tetherbot0, 120 links, 119 joints
Joints:
- joint gripper0_to_dockpoint0: origin xyz=0.0 0.0 0.143 rpy=0.0 -0.0 0.0 -> xyz=0.0 0.0 0.143 rpy=3.141592653589793 -0.0 0.0
- joint gripper1_to_dockpoint1: origin xyz=0.0 0.0 0.143 rpy=0.0 -0.0 0.0 -> xyz=0.0 0.0 0.143 rpy=3.141592653589793 -0.0 0.0
- joint gripper2_to_dockpoint2: origin xyz=0.0 0.0 0.143 rpy=0.0 -0.0 0.0 -> xyz=0.0 0.0 0.143 rpy=3.141592653589793 -0.0 0.0
- joint gripper3_to_dockpoint3: origin xyz=0.0 0.0 0.143 rpy=0.0 -0.0 0.0 -> xyz=0.0 0.0 0.143 rpy=3.141592653589793 -0.0 0.0
- joint gripper4_to_dockpoint4: origin xyz=0.0 0.0 0.143 rpy=0.0 -0.0 0.0 -> xyz=0.0 0.0 0.143 rpy=3.141592653589793 -0.0 0.0
